File: KiCad files/NDE.kicad_sch (KiCad schematic)
At the start: 2 parts, among them U1 LM7805_TO220

Commit message: Schematic layout
Parts:
- added C1, C3: 100n, symbol Device:C
- added C2, C4: 100u, symbol Device:C_Polarized
- added J1: Nabíjací modul, symbol Connector:Screw_Terminal_01x02
- added J2: Step-up input, symbol Connector:Screw_Terminal_01x02
- added J3: Step-up output, symbol Connector:Screw_Terminal_01x02
- added J6: Solenoid X, symbol Connector:Conn_01x02_Pin
- added J7: Solenoid Y, symbol Connector:Conn_01x02_Pin
- added JP1: +BATT default, symbol Jumper:Jumper_3_Open
Connections:
- net at BT1.N1: now also BT1.P2
- net GND: now reaches BT1.N2
- net GND: now also U1.2 (GND), C1.2, C2.2, C3.2, C4.2, J1.2 (Pin_2), J2.2 (Pin_2), J3.2 (Pin_2)
- net +BATT: now reaches BT1.P1
- net +BATT: now also U1.1 (VI), C1.1, C2.1, J1.1 (Pin_1), J2.1 (Pin_1), JP1.1 (A)
- net +5V: now reaches U1.3 (VO)
- net +5V: now also C3.1, C4.1
- new net H-mostík/VCC: JP1.2 (C)
- new net Vdrive: J3.1 (Pin_1), JP1.3 (B)
Other:
- added sheet BlackPill V3.0 (blackpill.kicad_sch)
- added sheet Gyroskop (gyro.kicad_sch)
- added sheet H-mostík (hbridge.kicad_sch)
- added sheet Magnetometer (magnetometer.kicad_sch)
- note added: "Baterka"
- note added: "DC/DC"
- note added: "Gyro"
- note added: "H-mostík"
- note added: "Magnetometer → mimo DPS"
- note added: "Nabíjací modul"
- note added: "Regulátor"
- note added: "STM"
- moved on the sheet: BT1, U1

Commit message: Board v1
Parts:
- removed J6: Solenoid X, symbol Connector:Conn_01x02_Pin
- removed J7: Solenoid Y, symbol Connector:Conn_01x02_Pin
- added JP2: Jumper_3_Open, Connector_PinHeader_2.54mm:PinHeader_1x03_P2.54mm_Vertical, symbol Jumper:Jumper_3_Open
- C1, C3: footprint (none) -> Capacitor_THT:C_Disc_D5.0mm_W2.5mm_P2.50mm
- C2, C4: value 100u -> 10u; footprint (none) -> Capacitor_THT:CP_Radial_D5.0mm_P2.50mm
- J1, J2, J3: footprint (none) -> TerminalBlock_Phoenix:TerminalBlock_Phoenix_MKDS-1,5-2_1x02_P5.00mm_Horizontal
- JP1: footprint (none) -> Connector_PinHeader_2.54mm:PinHeader_1x03_P2.54mm_Vertical
Connections:
- net +5V: now also JP2.3 (B)
- net GND: now also JP2.1 (A)
- net Vdrive renamed +10V
- new net Gyroskop/AD0: JP2.2 (C)
- no-connect marks 0 -> 35
Other:
- added sheet Solenoid X (solenoid.kicad_sch)
- added sheet Solenoid Y (solenoid.kicad_sch)
- sheet BlackPill V3.0 ports: added 3V3.0, 3V3.1, 5V.0, 5V.1, A0, A1, A10, A11, A12, A15, A2, A3, A4, A5, A6, A7, A8, A9, B0, B1, B10, B12, B13, B14, B15, B2, B3, B4, B5, B6, B7, B8, B9, C13, C14, C15, G.0, G.1, R, VB; removed none
- sheet Gyroskop ports: added AD0, GND, INT, SCL, SDA, VCC, XCL, XDA; removed none
- sheet Magnetometer ports: added DRDY, GND, SCL, SDA, VCC; removed none
- note added: "Prídavné konektory na externý DC/DC menič"
- note added: "na kábli"
- note added: "voliteľný"
- note removed: "Baterka"
- note removed: "DC/DC"
- note removed: "Gyro"
- note removed: "H-mostík"
- note removed: "Magnetometer → mimo DPS"
- note removed: "Nabíjací modul"
- note removed: "Regulátor"
- note removed: "STM"
- moved on the sheet: BT1, C1, C2, C3, C4, J1, J2, J3, JP1, U1
