File: KiCad files/blackpill.kicad_sch (KiCad schematic)
At the start: 0 parts

Commit message: Board v1
Parts:
- added J8, J9: Conn_01x20_Socket, Connector_PinSocket_2.54mm:PinSocket_1x20_P2.54mm_Vertical, symbol Connector:Conn_01x20_Socket
Connections:
- new net 3V3.0: J8.20 (Pin_20)
- new net 3V3.1: J9.3 (Pin_3)
- new net 5V.0: J8.18 (Pin_18)
- new net 5V.1: J9.1 (Pin_1)
- new net A0: J9.15 (Pin_15)
- new net A1: J9.14 (Pin_14)
- new net A10: J8.7 (Pin_7)
- new net A11: J8.8 (Pin_8)
- new net A12: J8.9 (Pin_9)
- new net A15: J8.10 (Pin_10)
- new net A2: J9.13 (Pin_13)
- new net A3: J9.12 (Pin_12)
- new net A4: J9.11 (Pin_11)
- new net A5: J9.10 (Pin_10)
- new net A6: J9.9 (Pin_9)
- new net A7: J9.8 (Pin_8)
- new net A8: J8.5 (Pin_5)
- new net A9: J8.6 (Pin_6)
- new net B0: J9.7 (Pin_7)
- new net B1: J9.6 (Pin_6)
- new net B10: J9.4 (Pin_4)
- new net B12: J8.1 (Pin_1)
- new net B13: J8.2 (Pin_2)
- new net B14: J8.3 (Pin_3)
- new net B15: J8.4 (Pin_4)
- new net B2: J9.5 (Pin_5)
- new net B3: J8.11 (Pin_11)
- new net B4: J8.12 (Pin_12)
- new net B5: J8.13 (Pin_13)
- new net B6: J8.14 (Pin_14)
- new net B7: J8.15 (Pin_15)
- new net B8: J8.16 (Pin_16)
- new net B9: J8.17 (Pin_17)
- new net C13: J9.19 (Pin_19)
- new net C14: J9.18 (Pin_18)
- new net C15: J9.17 (Pin_17)
- new net G.0: J8.19 (Pin_19)
- new net G.1: J9.2 (Pin_2)
- new net R: J9.16 (Pin_16)
- new net VB: J9.20 (Pin_20)
