File: KiCad files/hbridge.kicad_sch (KiCad schematic)
At the start: 2 parts

Commit message: Board v1
Parts:
- J4, J5: footprint (none) -> Connector_PinSocket_2.54mm:PinSocket_1x06_P2.54mm_Vertical
Changed lines of the file:
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@@
 	)
 	(symbol
-		(lib_name "Conn_01x06_Socket_1")
 		(lib_id "Connector:Conn_01x06_Socket")
 		(at 142.24 99.06 0)
@@
 		(on_board yes)
 		(dnp no)
-		(fields_autoplaced yes)
 		(property "Reference" "J4"
 			(at 143.51 99.6949 0)
@@
 			)
 		)
-		(property "Footprint" ""
+		(property "Footprint" "Connector_PinSocket_2.54mm:PinSocket_1x06_P2.54mm_Vertical"
 			(at 142.24 99.06 0)
 			(effects
@@
 			)
 		)
-		(property "Footprint" ""
+		(property "Footprint" "Connector_PinSocket_2.54mm:PinSocket_1x06_P2.54mm_Vertical"
 			(at 151.13 99.06 0)
 			(effects
